Commit message: fixed-base implmentation

File: resource/anymal_c/urdf/robot_3D.urdf (robot description, URDF)
Before this commit: robot 2DrobotArm, 5 links, 4 joints
Joints:
- removed joint link2Tolink3
- added joint link1Tolink3: type revolute, parent link2, child link3, origin xyz=0 0 0.3, axis 1 0 0
- joint link3Tolink4: axis 0 0 1 -> 0 1 0; limit lower=-0.1 upper=0.3 effort=80.0 velocity=7.5 -> (none)
